File: boards/SwellEncoder/SwellEncoder.sch (KiCad schematic (older format))
At the start: 8 parts, among them IC1 ATMEGA48-P

Commit message: First version of thumb encoder schematics
Connections:
- net at ISP.5: now also IC1.1 ((PCINT14/~RESET~)PC6), R1.2
Changed lines of the file:
@@
 Sheet 1 1
 Title ""
-Date "6 oct 2013"
+Date "13 oct 2013"
 Rev ""
 Comp ""
@@
 Wire Wire Line
 	3700 1150 3700 1000
+Connection ~ 3700 2000
 $EndSCHEMATC
