File: boards/MatrixShiftEncoder/MatrixShiftEncoder.sch (KiCad schematic (older format))
At the start: 61 parts

Commit message: Added old firmware and design files
Parts:
- removed U? (x16): 74LS151, ~, symbol 74LS151
- removed U? (x2): 74LS153, ~, symbol 74LS153
- added U? (x16): 4014, symbol 4014
Connections:
- net labels added: clk, str
- net labels removed: s0, s1, s2, s3, s4
- wire segments 479 -> 442
- no-connect marks 5 -> 4
Other:
- moved on the sheet: P?
