File: boards/KeyboardEncoder/KeyboardEncoder.kicad_pcb (KiCad board)
At the start: 2 copper layers, 0 parts

Commit message: PCB layout for keyboard scanner and piston encoder
Parts:
- added C1: 100nF, Capacitor_THT:C_Disc_D4.3mm_W1.9mm_P5.00mm, F.Cu at (221.1, 108.3)
- added C2: 100nF, Capacitor_THT:C_Disc_D4.3mm_W1.9mm_P5.00mm, F.Cu at (221.1, 111.8)
- added C3: C_Polarized, Capacitor_THT:CP_Radial_D10.0mm_P5.00mm, F.Cu at (223.0, 100.8)
- added D1: 1N4148, Diode_THT:D_DO-35_SOD27_P7.62mm_Horizontal, F.Cu at (192.6, 109.2)
- added J1: ISP, Connector_IDC:IDC-Header_2x05_P2.54mm_Vertical, F.Cu at (207.2, 64.7)
- added J2: Encoder, Connector_IDC:IDC-Header_2x10_P2.54mm_Vertical, F.Cu at (207.2, 87.1)
- added J3: MIDI Out, Connector_PinHeader_2.54mm:PinHeader_1x03_P2.54mm_Vertical, F.Cu at (221.8, 87.7)
- added J4: SelectRX, Connector_PinHeader_2.54mm:PinHeader_1x03_P2.54mm_Vertical, F.Cu at (226.5, 87.7)
- added J5: MIDI In, Connector_PinHeader_2.54mm:PinHeader_1x03_P2.54mm_Vertical, F.Cu at (231.1, 87.7)
- added J7: BoardCon, Connector_IDC:IDC-Header_2x05_P2.54mm_Vertical, F.Cu at (219.1, 64.7)
- added J8: PistonEncoder, Connector_IDC:IDC-Header_2x05_P2.54mm_Vertical, F.Cu at (231.1, 64.7)
- added R1: 10k, Resistor_THT:R_Axial_DIN0204_L3.6mm_D1.6mm_P2.54mm_Vertical, F.Cu at (215.5, 86.9)
- added R2: 220, Resistor_THT:R_Axial_DIN0204_L3.6mm_D1.6mm_P2.54mm_Vertical, F.Cu at (215.5, 90.1)
- added R3: 220, Resistor_THT:R_Axial_DIN0204_L3.6mm_D1.6mm_P2.54mm_Vertical, F.Cu at (215.5, 93.2)
- added R4: 220, Resistor_THT:R_Axial_DIN0204_L3.6mm_D1.6mm_P2.54mm_Vertical, F.Cu at (215.5, 96.4)
- added R5: 220, Resistor_THT:R_Axial_DIN0204_L3.6mm_D1.6mm_P2.54mm_Vertical, F.Cu at (215.5, 99.5)
- added RN1: 10k, Resistor_THT:R_Array_SIP9, F.Cu at (216.1, 83.2)
- added U1: ATmega48-20P, Package_DIP:DIP-28_W7.62mm, F.Cu at (192.7, 60.6)
- added U2: 6N138, Package_DIP:DIP-8_W7.62mm, F.Cu at (192.7, 97.8)
