File: boards/TechnicsEncoder/TechnicsEncoder.kicad_pcb (KiCad board)
At the start: 2 copper layers, 0 parts

Commit message: Using custom TO220 cooler, fixed and finished several PCBs
Parts:
- added C1: 100nF, Capacitor_THT:C_Disc_D4.3mm_W1.9mm_P5.00mm, F.Cu at (130.8, 98.8)
- added C2: 100nF, Capacitor_THT:C_Disc_D4.3mm_W1.9mm_P5.00mm, F.Cu at (153.2, 80.3)
- added C5: 33uF, Capacitor_THT:CP_Radial_D7.5mm_P2.50mm, F.Cu at (170.5, 109.7)
- added C6: 10uF, Capacitor_THT:CP_Radial_D6.3mm_P2.50mm, F.Cu at (171.8, 71.0)
- added C7: 100nF, Capacitor_THT:C_Disc_D4.3mm_W1.9mm_P5.00mm, F.Cu at (115.6, 71.5)
- added D1: 1N4148, Diode_THT:D_DO-35_SOD27_P7.62mm_Horizontal, F.Cu at (100.3, 68.3)
- added H1: MountingHole, MountingHole:MountingHole_3mm, F.Cu at (181.7, 69.8)
- added H2: MountingHole, MountingHole:MountingHole_3mm, F.Cu at (181.7, 112.8)
- added H3: MountingHole, MountingHole:MountingHole_3mm, F.Cu at (80.7, 69.8)
- added H4: MountingHole, MountingHole:MountingHole_3mm, F.Cu at (80.7, 112.8)
- added HS1: Heatsink_Pad, Custom_Heatsinks:Heatsink_Aavid_TO-220_H12.7mm, F.Cu at (160.5, 92.0)
- added J1: ISP, Connector_IDC:IDC-Header_2x05_P2.54mm_Vertical, F.Cu at (128.8, 109.7)
- added J2: Bender, Connector_PinHeader_2.54mm:PinHeader_1x03_P2.54mm_Vertical, F.Cu at (104.9, 112.3)
- added J3: Technics, Connector_JST:JST_PH_B15B-PH-K_1x15_P2.00mm_Vertical, F.Cu at (80.6, 77.9)
- added J4: SelectRX, Connector_PinHeader_2.54mm:PinHeader_1x03_P2.54mm_Vertical, F.Cu at (162.1, 69.3)
- added J5: MIDI In, Connector_PinHeader_2.54mm:PinHeader_1x03_P2.54mm_Vertical, F.Cu at (89.7, 68.3)
- added J6: MIDI Out, Connector_PinHeader_2.54mm:PinHeader_1x03_P2.54mm_Vertical, F.Cu at (127.8, 73.9)
- added J7: BoardCon, Connector_IDC:IDC-Header_2x05_P2.54mm_Vertical, F.Cu at (158.8, 109.7)
- added J8: PistonEncoder, Connector_IDC:IDC-Header_2x05_P2.54mm_Vertical, F.Cu at (179.1, 85.9)
- added R1: 2k2, Resistor_THT:R_Axial_DIN0204_L3.6mm_D1.6mm_P2.54mm_Vertical, F.Cu at (119.4, 71.4)
- added R2: 220, Resistor_THT:R_Axial_DIN0204_L3.6mm_D1.6mm_P7.62mm_Horizontal, F.Cu at (153.7, 104.1)
- added R3: 220, Resistor_THT:R_Axial_DIN0204_L3.6mm_D1.6mm_P7.62mm_Horizontal, F.Cu at (146.1, 98.3)
- added R4: 220, Resistor_THT:R_Axial_DIN0204_L3.6mm_D1.6mm_P2.54mm_Vertical, F.Cu at (94.8, 68.3)
- added R5: 220, Resistor_THT:R_Axial_DIN0204_L3.6mm_D1.6mm_P7.62mm_Horizontal, F.Cu at (140.9, 69.6)
- added R6: 220, Resistor_THT:R_Axial_DIN0204_L3.6mm_D1.6mm_P2.54mm_Vertical, F.Cu at (123.2, 73.9)
- added RN1: R_Pack04, Resistor_THT:R_Array_SIP8, F.Cu at (103.4, 87.9)
- added RN2: R_Pack04, Resistor_THT:R_Array_SIP8, F.Cu at (103.7, 96.0)
- added RN3: R_Pack04, Resistor_THT:R_Array_SIP8, F.Cu at (103.6, 103.9)
- added U1: ATmega48-20P, Package_DIP:DIP-28_W7.62mm, F.Cu at (151.1, 87.9)
- added U2: 6N137, Package_DIP:DIP-8_W7.62mm, F.Cu at (104.9, 68.8)
- added U3: 74LS14, Package_DIP:DIP-14_W7.62mm, F.Cu at (148.6, 72.6)
- added U4: L7805, Package_TO_SOT_THT:TO-220-3_Vertical, F.Cu at (164.1, 94.5)
Routing:
- net +5V: track 0.00 -> 253.3 mm, vias 0 -> 2
- net +12V: track 0.00 -> 74.3 mm, vias 0 -> 2
- net MIDI Rx: track 0.00 -> 69.0 mm
- net Read: track 0.00 -> 67.5 mm, vias 0 -> 2
- net MISO: track 0.00 -> 59.3 mm
- net Reset: track 0.00 -> 57.2 mm, vias 0 -> 4
- net SCK: track 0.00 -> 56.3 mm
- net Bend: track 0.00 -> 55.8 mm
- net TXD_OUT: track 0.00 -> 47.5 mm, vias 0 -> 4
- net SDA: track 0.00 -> 46.8 mm, vias 0 -> 2
- net D0: track 0.00 -> 44.7 mm, vias 0 -> 2
- net SCL: track 0.00 -> 44.7 mm
- net Latch: track 0.00 -> 44.3 mm, vias 0 -> 2
- net MOSI: track 0.00 -> 42.6 mm, vias 0 -> 2
- net Net-(J4-Pin_3): track 0.00 -> 40.1 mm, vias 0 -> 2
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- added copper zone on B.Cu, net GND
Other:
- board outline added: 110.5 x 52.6 mm
