File: boards/PedalEncoder/PedalEncoder.kicad_pcb (KiCad board)
At the start: 2 copper layers, 125 x 38.5 mm, 35 parts, among them J1 Pwr, J2 Control, J3 Switch, J4 ISP, J5 Pedal, J6 MIDI Out, J7 I2C, Q1 BC547, Q2 BC547, U1 4069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

Commit message: Fixed PedalEncoder ISP connections
Parts:
- moved RN1 3.34 mm to (148.1, 87.6)
- moved C1 2.54 mm to (123.4, 87.9)
- moved Q1 1.52 mm to (161.5, 81.3)
Connections:
- RN1 pad 3: Net-(J5-Pin_8) -> Net-(J5-Pin_5)
- RN1 pad 4: Net-(J5-Pin_6) -> Net-(J5-Pin_3)
- RN1 pad 5: Net-(J5-Pin_5) -> MOSI
- RN1 pad 6: Net-(J5-Pin_3) -> MISO
- RN1 pad 7: MOSI -> Net-(J5-Pin_8)
- RN1 pad 8: MISO -> SCK
- RN1 pad 9: SCK -> Net-(J5-Pin_6)
Routing:
- net MOSI: track 9.65 -> 111.2 mm, vias 0 -> 6
- net SCK: track 151.1 -> 99.5 mm, vias 4 -> 2
- net Net-(J5-Pin_10): track 96.7 -> 53.9 mm
- net Net-(J5-Pin_8): track 62.5 -> 36.3 mm
- net Net-(J5-Pin_6): track 55.9 -> 33.7 mm, vias 2 -> 0
- net GND: track 54.3 -> 39.3 mm, vias 10 -> 8
- net MISO: track 86.6 -> 91.2 mm
- net Net-(J5-Pin_7): track 26.5 -> 23.1 mm
- net Net-(Q1-B): track 26.1 -> 23.4 mm
- net Net-(J5-Pin_3): track 9.65 -> 11.9 mm
- net Net-(J5-Pin_5): track 9.65 -> 11.6 mm
- net +5V: track 251.3 -> 253.1 mm, vias 4 -> 2
- net Net-(U2-PD5): track 27.4 -> 25.8 mm
- net LED: track 8.64 -> 10.2 mm
- net Reset: track 89.4 -> 88.4 mm
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