File: boards/LEDController/LEDController.kicad_sch (KiCad schematic)
At the start: 16 parts, among them J1 ISP, J2 LED1, J3 LED2, J4 Buttons, J5 BoardCon, J6 BoardConOut, J7 LED3, U1 ULN2803A, U2 ATmega48-20P, U4 ULN2803A

Commit message: Exported LEDController gerber
Parts:
- J4: footprint Connector_PinSocket_2.54mm:PinSocket_2x05_P2.54mm_Vertical -> Connector_PinHeader_2.54mm:PinHeader_2x05_P2.54mm_Vertical
- J7: footprint Connector_PinSocket_2.54mm:PinSocket_1x02_P2.54mm_Vertical -> Connector_PinHeader_2.54mm:PinHeader_1x02_P2.54mm_Vertical
Changed lines of the file:
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@@
 	)
 	(junction
+		(at 233.68 86.36)
+		(diameter 0)
+		(color 0 0 0 0)
+	)
+	(junction
 		(at 233.68 97.79)
 		(diameter 0)
@@
 	(wire
 		(pts
+			(xy 220.98 86.36) (xy 233.68 86.36)
+		)
+		(stroke
+			(width 0)
+			(type default)
+		)
+	)
+	(wire
+		(pts
 			(xy 63.5 135.89) (xy 63.5 139.7)
 		)
@@
 	(wire
 		(pts
-			(xy 233.68 83.82) (xy 233.68 95.25)
+			(xy 233.68 83.82) (xy 233.68 86.36)
 		)
 		(stroke
@@
 	(wire
 		(pts
+			(xy 233.68 86.36) (xy 233.68 95.25)
+		)
+		(stroke
+			(width 0)
+			(type default)
+		)
+	)
+	(wire
+		(pts
 			(xy 231.14 140.97) (xy 233.68 140.97)
 		)
@@
 	(wire
 		(pts
+			(xy 220.98 83.82) (xy 220.98 86.36)
+		)
+		(stroke
+			(width 0)
+			(type default)
+		)
+	)
+	(wire
+		(pts
 			(xy 241.3 83.82) (xy 241.3 86.36)
 		)
@@
 			)
 		)
-		(property "Footprint" "Connector_PinSocket_2.54mm:PinSocket_2x05_P2.54mm_Vertical"
+		(property "Footprint" "Connector_PinHeader_2.54mm:PinHeader_2x05_P2.54mm_Vertical"
 			(at 105.41 72.39 0)
 			(effects
@@
 			)
 		)
-		(property "Footprint" "Connector_PinSocket_2.54mm:PinSocket_1x02_P2.54mm_Vertical"
+		(property "Footprint" "Connector_PinHeader_2.54mm:PinHeader_1x02_P2.54mm_Vertical"
 			(at 142.24 167.64 0)
 			(effects
@@
 					(unit 1)
 				)
+			)
+		)
+	)
+	(symbol
+		(lib_id "power:PWR_FLAG")
+		(at 220.98 83.82 0)
+		(unit 1)
+		(exclude_from_sim no)
+		(in_bom yes)
+		(on_board yes)
+		(dnp no)
+		(fields_autoplaced yes)
+		(property "Reference" "#FLG03"
+			(at 220.98 81.915 0)
+			(effects
+				(font
+					(size 1.27 1.27)
+				)
+				(hide yes)
+			)
+		)
+		(property "Value" "PWR_FLAG"
+			(at 220.98 78.74 0)
+			(effects
+				(font
+					(size 1.27 1.27)
+				)
+			)
+		)
+		(property "Footprint" ""
+			(at 220.98 83.82 0)
+			(effects
+				(font
+					(size 1.27 1.27)
+				)
+				(hide yes)
+			)
+		)
+		(property "Datasheet" "~"
+			(at 220.98 83.82 0)
+			(effects
+				(font
+					(size 1.27 1.27)
+				)
+				(hide yes)
+			)
+		)
+		(property "Description" "Special symbol for telling ERC where power comes from"
+			(at 220.98 83.82 0)
+			(effects
+				(font
+					(size 1.27 1.27)
+				)
+				(hide yes)
+			)
+		)
+		(pin "1"
+		)
+		(instances
+			(project "LEDController"
+				(path "/75af7309-2f58-4fd2-89b0-eb551d087b2d"
+					(reference "#FLG03")
+					(unit 1)
+				)

Commit message: Fixed LEDController button header layout
Connections:
- net GND: now also J4.1 (Pin_1), J4.3 (Pin_3), J4.5 (Pin_5), J4.7 (Pin_7), J4.9 (Pin_9); no longer J4.10 (Pin_10), J4.2 (Pin_2), J4.4 (Pin_4), J4.6 (Pin_6), J4.8 (Pin_8)
- net MISO: now also J4.10 (Pin_10); no longer J4.9 (Pin_9)
- net MOSI: now also J4.4 (Pin_4); no longer J4.3 (Pin_3)
- net at U2.14 (PB0): now also J4.2 (Pin_2); no longer J4.1 (Pin_1)
- net at U2.15 (PB1): now also J4.8 (Pin_8); no longer J4.7 (Pin_7)
- net at U2.16 (PB2): now also J4.6 (Pin_6); no longer J4.5 (Pin_5)
Changed lines of the file:
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@@
-	(wire
-		(pts
-			(xy 97.79 69.85) (xy 97.79 64.77)
-		)
-		(stroke
-			(width 0)
-			(type default)
-		)
-	)
 	(wire
 		(pts
@@
 	(wire
 		(pts
+			(xy 93.98 74.93) (xy 100.33 74.93)
+		)
+		(stroke
+			(width 0)
+			(type default)
+		)
+	)
+	(wire
+		(pts
 			(xy 229.87 53.34) (xy 232.41 53.34)
 		)
@@
 	(wire
 		(pts
-			(xy 100.33 74.93) (xy 93.98 74.93)
-		)
-		(stroke
-			(width 0)
-			(type default)
-		)
-	)
-	(wire
-		(pts
 			(xy 105.41 115.57) (xy 104.14 115.57)
 		)
@@
 		(pts
 			(xy 88.9 123.19) (xy 88.9 165.1)
+		)
+		(stroke
+			(width 0)
+			(type default)
+		)
+	)
+	(wire
+		(pts
+			(xy 97.79 64.77) (xy 97.79 69.85)
 		)
 		(stroke
@@
 	(symbol
 		(lib_id "Connector_Generic:Conn_02x05_Odd_Even")
-		(at 105.41 72.39 0)
+		(at 107.95 72.39 0)
+		(mirror y)
 		(unit 1)
 		(exclude_from_sim no)
@@
 		(on_board yes)
 		(dnp no)
-		(fields_autoplaced yes)
 		(property "Reference" "J4"
 			(at 106.68 60.96 0)
@@
 		)
 		(property "Footprint" "Connector_PinHeader_2.54mm:PinHeader_2x05_P2.54mm_Vertical"
-			(at 105.41 72.39 0)
+			(at 107.95 72.39 0)
 			(effects
 				(font
@@
 		)
 		(property "Datasheet" "~"
-			(at 105.41 72.39 0)
+			(at 107.95 72.39 0)
 			(effects
 				(font
@@
 		)
 		(property "Description" "Generic connector, double row, 02x05, odd/even pin numbering scheme (row 1 odd numbers, row 2 even numbers), script generated (kicad-library-utils/schlib/autogen/connector/)"
-			(at 105.41 72.39 0)
-			(effects
-				(font
+			(at 107.95 72.39 0)
+			(effects
+				(font
