File: boards/MIDIController/MIDIController.kicad_pcb (KiCad board)
At the start: 2 copper layers, 150 x 100 mm, 39 parts, among them J1 VBAT, J10 RJ45_Bel_SI-60062-F_fixed, J11 USB, J2 MIDICon, J3 IO_Boards, J4 USB_A, J5 I2S1, J6 I2S2, J7 Raspberry_Pi_2_3, J8 RPI_Pwr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

Commit message: Added line jacks for the audio board.
Parts:
- removed H5: MountingHole, MountingHole:MountingHole_2.7mm_M2.5
- added J12: LineIn, Custom_Connectors:Jack_3.5mm_Ledino_KB3SPRS_Horizontal_Stereo, F.Cu at (87.6, 139.2)
- added J13: LineOut, Custom_Connectors:Jack_3.5mm_Ledino_KB3SPRS_Horizontal_Stereo, F.Cu at (102.0, 139.2)
- added J14: Conn_02x05_Odd_Even, Connector_PinHeader_2.54mm:PinHeader_2x05_P2.54mm_Vertical, F.Cu at (107.8, 122.4)
- J1: value VBAT -> Bat; footprint Connector_PinHeader_2.54mm:PinHeader_1x01_P2.54mm_Vertical -> Connector_PinHeader_2.54mm:PinHeader_1x02_P2.54mm_Vertical
- R9: value 4k7 -> 470
- moved C2 102.9 mm to (212.6, 128.7), turned to 180 degrees
- moved C1 95.9 mm to (199.9, 142.0), turned to 90 degrees
- moved J1 2.29 mm to (164.1, 87.1), turned to 180 degrees
- moved R9 0.63 mm to (75.9, 53.1)
Connections:
- J1 pad 1: Net-(BT1-+) -> GND
Routing:
- net Net-(J14-Pin_2): track 0.00 -> 61.6 mm
- net Net-(J14-Pin_1): track 0.00 -> 53.8 mm
- net Net-(J14-Pin_3): track 0.00 -> 34.2 mm
- net Net-(J14-Pin_5): track 0.00 -> 18.8 mm
- net +5V: track 366.5 -> 349.3 mm
- net Net-(J14-Pin_9): track 0.00 -> 10.5 mm
- net +3.3V: track 173.4 -> 170.0 mm
- net /TXD1: track 191.7 -> 193.7 mm
- net /TXD5: track 168.4 -> 170.2 mm
- net /TXD4: track 159.6 -> 161.4 mm
- net /I2S_OUT2: track 93.4 -> 92.6 mm
- net /SDA: track 305.6 -> 304.9 mm
- net /RPI_SCLK: track 108.6 -> 108.0 mm
- net /RPI_MOSI: track 109.8 -> 109.2 mm
- net /Int_RPI: track 108.6 -> 108.0 mm
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